File: REVA/open-lux-A.brd (EAGLE design)
At the start: 52.4 x 52.7 mm, 52 parts, among them IC1 ATMEGA328P, IC2 MCP73831, IC4 MCP1700-33, J1 AYZ0202, Q4 BSS123, Q5 BSS123, Q6 BSS123, Q7 BSS123, X1 USBSMD

Commit message: update
Parts:
- renumbered J2 to LCDLIGHT
Other:
- board text added: "A0"
- board text added: "A1"
- board text added: "GND"
- board text added: "NOKIA 5110"
- board text added: "RX"
- board text added: "SCL"
- board text added: "SDA"
- board text added: "TX"
- board text added: "VCC"
Changed lines of the file:
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@@
 <layer number="23" name="tOrigins" color="15" fill="1" visible="yes" active="yes"/>
 <layer number="24" name="bOrigins" color="15" fill="1" visible="yes" active="yes"/>
-<layer number="25" name="tNames" color="7" fill="1" visible="yes" active="yes"/>
+<layer number="25" name="tNames" color="7" fill="1" visible="no" active="yes"/>
 <layer number="26" name="bNames" color="7" fill="1" visible="yes" active="yes"/>
 <layer number="27" name="tValues" color="7" fill="1" visible="no" active="yes"/>
@@
 <text x="42.926" y="49.276" size="1.27" layer="21" rot="R315">OPEN-LUX</text>
 <text x="50.546" y="44.958" size="0.8128" layer="21" rot="R135">REVA</text>
+<text x="37.846" y="46.482" size="0.8128" layer="21" rot="R270">GND</text>
+<text x="18.796" y="41.91" size="0.8128" layer="22" rot="MR270">GND</text>
+<text x="49.53" y="13.97" size="0.8128" layer="22" rot="MR0">GND</text>
+<text x="26.67" y="42.926" size="0.8128" layer="22" rot="MR0">NOKIA 5110</text>
+<text x="21.336" y="42.418" size="0.8128" layer="22" rot="MR270">VCC</text>
+<text x="23.622" y="41.91" size="0.8128" layer="22" rot="MR270">RX</text>
+<text x="26.416" y="39.116" size="0.8128" layer="22" rot="MR270">TX</text>
+<text x="28.702" y="38.862" size="0.8128" layer="22" rot="MR270">SDA</text>
+<text x="31.75" y="43.18" size="0.8128" layer="22" rot="MR270">SCL</text>
+<text x="34.036" y="39.878" size="0.8128" layer="22" rot="MR270">A0</text>
+<text x="36.576" y="41.402" size="0.8128" layer="22" rot="MR270">A1</text>
+<wire x1="37.338" y1="40.386" x2="40.386" y2="40.386" width="0.4064" layer="22"/>
+<wire x1="40.386" y1="40.386" x2="40.386" y2="50.292" width="0.4064" layer="22"/>
+<wire x1="17.526" y1="40.386" x2="15.494" y2="40.386" width="0.4064" layer="22"/>
+<wire x1="40.386" y1="50.546" x2="38.354" y2="50.546" width="0.4064" layer="22"/>
+<wire x1="38.354" y1="50.546" x2="39.116" y2="51.308" width="0.4064" layer="22"/>
+<wire x1="38.354" y1="50.546" x2="39.116" y2="49.784" width="0.4064" layer="22"/>
+<wire x1="15.494" y1="40.386" x2="15.494" y2="50.292" width="0.4064" layer="22"/>
+<wire x1="15.494" y1="50.292" x2="16.764" y2="50.292" width="0.4064" layer="22"/>
+<wire x1="16.764" y1="50.292" x2="16.002" y2="51.054" width="0.4064" layer="22"/>
+<wire x1="16.764" y1="50.292" x2="16.256" y2="49.784" width="0.4064" layer="22"/>
 </plain>
 <attributes>
@@
 </element>
 <element name="BTN" library="adafruit" package="EVQ-Q2" value="" x="5.715" y="25.4" smashed="yes">
-<attribute name="NAME" x="0.175" y="25.09" size="1.27" layer="25"/>
+<attribute name="NAME" x="4.397" y="25.964" size="1.27" layer="25" rot="R180"/>
 <attribute name="VALUE" x="2.515" y="20.6" size="1.27" layer="27"/>
 </element>
@@
 <attribute name="VALUE" x="53.34" y="40.005" size="1.27" layer="27" rot="R90"/>
 </element>
-<element name="J2" library="jumper" package="JP1" value="" x="13.335" y="49.53" smashed="yes" rot="R90">
-<attribute name="NAME" x="14.097" y="51.943" size="0.8128" layer="25" ratio="10" rot="R180"/>
+<element name="LCDLIGHT" library="jumper" package="JP1" value="" x="13.335" y="49.53" smashed="yes" rot="R90">
+<attribute name="NAME" x="16.383" y="52.197" size="0.8128" layer="25" ratio="10" rot="R180"/>
 <attribute name="VALUE" x="15.875" y="52.451" size="1.27" layer="27" ratio="10" rot="R180"/>
 </element>
@@
 <contactref element="SV2" pad="2"/>
 <contactref element="THM1" pad="2"/>
-<contactref element="J2" pad="1"/>
+<contactref element="LCDLIGHT" pad="1"/>
 <contactref element="RIR4" pad="2"/>
 <contactref element="RIR3" pad="2"/>
@@
 <signal name="N$8">
 <contactref element="N1" pad="7"/>
-<contactref element="J2" pad="2"/>
+<contactref element="LCDLIGHT" pad="2"/>
 <wire x1="13.97" y1="51.308" x2="12.192" y2="49.53" width="0.254" layer="1"/>
 <wire x1="15.24" y1="51.308" x2="13.97" y2="51.308" width="0.254" layer="1"/>

Commit message: update
Parts:
- removed R14, R15: 10K, adafruit:R0805
Connections:
- net +3V3: no longer C14.1, LUXNIR.VDD, R14.2, R15.2
- net SCL: no longer R15.1
- net SDA: no longer R14.1
- net VCC: now also C14.1, LUXNIR.VDD
Routing:
- net GREEN: track 149.1 -> 84.2 mm, vias 7 -> 5
- net MOSI: track 19.9 -> 75.6 mm, vias 1 -> 3
- net RED: track 94.6 -> 142.5 mm, vias 5 -> 9
- net +3V3: track 47.2 -> 9.28 mm, vias 7 -> 2
- net D2: track 25.6 -> 60.3 mm, vias 2 -> 4
- net TXD: track 39.6 -> 73.9 mm, vias 2 -> 4
- net SDA: track 95.2 -> 65.2 mm, vias 10 -> 4
- net GND: track 299.6 -> 324.6 mm, vias 9 -> 10
- net D5: track 67.6 -> 43.9 mm, vias 3 -> 5
- net VBAT: track 73.7 -> 97.1 mm, vias 5 -> 4
- net BLUE: track 89.5 -> 66.3 mm
- net VDD: track 71.5 -> 53.3 mm, vias 4 -> 5
- net VCC: track 187.0 -> 169.7 mm, vias 6 -> 3
- net RESET: track 57.6 -> 73.8 mm, vias 4 -> 3
- net D3: track 50.1 -> 34.9 mm, vias 2 -> 3
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Other:
- board text added: "LUX"
- board text added: "RGB"
