File: REVA/open-lux-A.brd (EAGLE design)
At the start: 52.4 x 52.7 mm, 50 parts, among them IC1 ATMEGA328P, IC2 MCP73831, IC4 MCP1700-33, J1 AYZ0202, Q4 BSS123, Q5 BSS123, Q6 BSS123, Q7 BSS123, X1 USBSMD

Commit message: update
Connections:
- removed net +3V3: C15.1, LUXRGB.1
- net VCC: now also C15.1, LUXRGB.1
Routing:
- net GND: track 324.6 -> 0.00 mm, vias 10 -> 0
- net VCC: track 169.7 -> 0.00 mm, vias 3 -> 0
- net RED: track 142.5 -> 0.00 mm, vias 9 -> 0
- net VBAT: track 97.1 -> 0.00 mm, vias 4 -> 0
- net GREEN: track 84.2 -> 0.00 mm, vias 5 -> 0
- net MOSI: track 75.6 -> 0.00 mm, vias 3 -> 0
- net TXD: track 73.9 -> 0.00 mm, vias 4 -> 0
- net RESET: track 73.8 -> 0.00 mm, vias 3 -> 0
- net BLUE: track 66.3 -> 0.00 mm, vias 6 -> 0
- net SDA: track 65.2 -> 0.00 mm, vias 4 -> 0
- net D2: track 60.3 -> 0.00 mm, vias 4 -> 0
- net A0: track 56.5 -> 0.00 mm, vias 3 -> 0
- net VDD: track 53.3 -> 0.00 mm, vias 5 -> 0
- net VBUS: track 51.9 -> 0.00 mm, vias 4 -> 0
- net A1: track 49.7 -> 0.00 mm, vias 2 -> 0
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