File: REVA/open-lux-A.sch (EAGLE design)
At the start: 52 parts, among them IC1 ATMEGA328P, IC2 MCP73831, IC4 MCP1700-33, J1 AYZ0202, Q4 BSS123, Q5 BSS123, Q6 BSS123, Q7 BSS123, X1 USBSMD

Commit message: update
Parts:
- renumbered J2 to LCDLIGHT
Changed lines of the file:
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@@
 <part name="THM1" library="adafruit" deviceset="1X2" device="-3.5MM"/>
 <part name="RTHM1" library="rcl" deviceset="R-US_" device="R0805" value="3k"/>
-<part name="J2" library="jumper" deviceset="JP1E" device=""/>
+<part name="LCDLIGHT" library="jumper" deviceset="JP1E" device=""/>
 <part name="RIR3" library="rcl" deviceset="R-EU_" device="R0805" value="10K"/>
 <part name="RIR4" library="rcl" deviceset="R-EU_" device="R0805" value="10K"/>
@@
 <attribute name="VALUE" x="265.176" y="-5.334" size="1.778" layer="96"/>
 </instance>
-<instance part="J2" gate="A" x="475.996" y="137.16" rot="R180"/>
+<instance part="LCDLIGHT" gate="A" x="475.996" y="137.16" rot="R180"/>
 <instance part="RIR3" gate="G$1" x="208.28" y="147.32" smashed="yes" rot="R90">
 <attribute name="NAME" x="212.09" y="147.32" size="1.778" layer="95"/>
@@
 <pinref part="P+11" gate="VCC" pin="VCC"/>
 <wire x1="485.902" y1="138.684" x2="486.664" y2="140.97" width="0.1524" layer="91"/>
-<pinref part="J2" gate="A" pin="1"/>
+<pinref part="LCDLIGHT" gate="A" pin="1"/>
 <wire x1="475.996" y1="139.7" x2="485.902" y2="138.684" width="0.1524" layer="91"/>
 </segment>
@@
 <pinref part="N1" gate="1" pin="7"/>
 <wire x1="423.926" y1="140.97" x2="473.71" y2="142.24" width="0.1524" layer="91"/>
-<pinref part="J2" gate="A" pin="2"/>
+<pinref part="LCDLIGHT" gate="A" pin="2"/>
 <wire x1="473.71" y1="142.24" x2="473.456" y2="139.7" width="0.1524" layer="91"/>
 </segment>

Commit message: update
Parts:
- removed R14, R15: 10K, adafruit:R-US_R0805
Connections:
- net +3V3: no longer C14.1, LUXNIR.3.3V, R14.2, R15.2
- net SCL: no longer R15.1
- net SDA: no longer R14.1
- net VCC: now also C14.1, LUXNIR.3.3V
Changed lines of the file:
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@@
 <setting verticaltext="up"/>
 </settings>
-<grid distance="0.1" unitdist="inch" unit="inch" style="lines" multiple="1" display="no" altdistance="0.01" altunitdist="inch" altunit="inch"/>
+<grid distance="0.01" unitdist="inch" unit="inch" style="lines" multiple="1" display="no" altdistance="0.01" altunitdist="inch" altunit="inch"/>
 <layers>
 <layer number="1" name="Top" color="4" fill="1" visible="no" active="no"/>
@@
 <part name="U$2" library="microbuilder" deviceset="GND" device=""/>
 <part name="C14" library="adafruit" deviceset="C-US" device="C0805" value="0.1uF"/>
-<part name="R14" library="adafruit" deviceset="R-US_" device="R0805" value="10K"/>
-<part name="R15" library="adafruit" deviceset="R-US_" device="R0805" value="10K"/>
 <part name="LUXRGB" library="dwbLibrary" deviceset="TCS34725" device=""/>
 <part name="U$3" library="microbuilder" deviceset="GND" device=""/>
 <part name="C15" library="adafruit" deviceset="C-US" device="C0805" value="0.1uF"/>
 <part name="+3V8" library="supply1" deviceset="+3V3" device=""/>
-<part name="+3V15" library="supply1" deviceset="+3V3" device=""/>
-<part name="+3V16" library="supply1" deviceset="+3V3" device=""/>
 <part name="N1" library="con-lstb" deviceset="MA08-1" device=""/>
 <part name="P+11" library="supply1" deviceset="VCC" device=""/>
@@
 <part name="IRP" library="SparkFun-Connectors" deviceset="M01" device="PTH"/>
 <part name="IRG" library="SparkFun-Connectors" deviceset="M01" device="PTH"/>
+<part name="P+3" library="supply1" deviceset="VCC" device=""/>
 </parts>
 <sheets>
@@
 <instance part="U$2" gate="G$1" x="298.704" y="62.738"/>
 <instance part="C14" gate="G$1" x="326.644" y="80.518"/>
-<instance part="R14" gate="G$1" x="263.144" y="103.378" rot="R90"/>
-<instance part="R15" gate="G$1" x="273.304" y="103.378" rot="R90"/>
 <instance part="LUXRGB" gate="G$1" x="382.016" y="-25.908"/>
 <instance part="U$3" gate="G$1" x="364.236" y="-56.388"/>
 <instance part="C15" gate="G$1" x="399.796" y="-23.368"/>
 <instance part="+3V8" gate="G$1" x="364.236" y="9.652"/>
-<instance part="+3V15" gate="G$1" x="298.704" y="98.298"/>
-<instance part="+3V16" gate="G$1" x="268.224" y="116.078"/>
 <instance part="N1" gate="1" x="416.306" y="133.35"/>
 <instance part="P+11" gate="VCC" x="486.664" y="143.51"/>
@@
 <instance part="IRP" gate="G$1" x="226.06" y="121.92"/>
 <instance part="IRG" gate="G$1" x="226.06" y="109.22"/>
+<instance part="P+3" gate="VCC" x="304.8" y="101.854"/>
 </instances>
 <busses>
@@
 <pinref part="IRP" gate="G$1" pin="1"/>
 </segment>
+<segment>
+<wire x1="303.784" y1="75.438" x2="298.704" y2="75.438" width="0.1524" layer="91"/>
+<wire x1="298.704" y1="75.438" x2="298.704" y2="90.678" width="0.1524" layer="91"/>
+<wire x1="326.644" y1="83.058" x2="326.644" y2="90.678" width="0.1524" layer="91"/>
+<wire x1="326.644" y1="90.678" x2="305.054" y2="90.678" width="0.1524" layer="91"/>
+<pinref part="LUXNIR" gate="G$1" pin="3.3V"/>
+<pinref part="C14" gate="G$1" pin="1"/>
+<pinref part="P+3" gate="VCC" pin="VCC"/>
+<wire x1="305.054" y1="90.678" x2="298.704" y2="90.678" width="0.1524" layer="91"/>
+<wire x1="304.8" y1="99.314" x2="305.054" y2="96.52" width="0.1524" layer="91"/>
+<wire x1="305.054" y1="96.52" x2="305.054" y2="90.678" width="0.1524" layer="91"/>
+</segment>
 </net>
 <net name="AREF" class="0">
@@
 <net name="SDA" class="0">
 <segment>
-<wire x1="263.144" y1="85.598" x2="263.144" y2="98.298" width="0.1524" layer="91"/>
 <wire x1="263.144" y1="85.598" x2="303.784" y2="85.598" width="0.1524" layer="91"/>
 <label x="288.544" y="85.598" size="1.778" layer="95"/>
-<pinref part="R14" gate="G$1" pin="1"/>
 <pinref part="LUXNIR" gate="G$1" pin="SDA"/>
 </segment>
@@
 <net name="SCL" class="0">
 <segment>
-<wire x1="273.304" y1="83.058" x2="273.304" y2="98.298" width="0.1524" layer="91"/>
 <wire x1="303.784" y1="83.058" x2="273.304" y2="83.058" width="0.1524" layer="91"/>
 <label x="288.544" y="83.058" size="1.778" layer="95"/>
 <pinref part="LUXNIR" gate="G$1" pin="SCL"/>
-<pinref part="R15" gate="G$1" pin="1"/>
 </segment>
 <segment>
@@
 <pinref part="+3V8" gate="G$1" pin="+3V3"/>
 </segment>
-<segment>
-<wire x1="298.704" y1="90.678" x2="298.704" y2="95.758" width="0.1524" layer="91"/>
-<wire x1="303.784" y1="75.438" x2="298.704" y2="75.438" width="0.1524" layer="91"/>
-<wire x1="298.704" y1="75.438" x2="298.704" y2="90.678" width="0.1524" layer="91"/>
-<wire x1="326.644" y1="83.058" x2="326.644" y2="90.678" width="0.1524" layer="91"/>
-<wire x1="326.644" y1="90.678" x2="298.704" y2="90.678" width="0.1524" layer="91"/>
-<junction x="298.704" y="90.678"/>
-<pinref part="LUXNIR" gate="G$1" pin="3.3V"/>
-<pinref part="C14" gate="G$1" pin="1"/>
-<pinref part="+3V15" gate="G$1" pin="+3V3"/>
-</segment>
-<segment>
-<wire x1="263.144" y1="108.458" x2="268.224" y2="108.458" width="0.1524" layer="91"/>
-<wire x1="268.224" y1="108.458" x2="268.224" y2="113.538" width="0.1524" layer="91"/>
-<wire x1="273.304" y1="108.458" x2="268.224" y2="108.458" width="0.1524" layer="91"/>
-<junction x="268.224" y="108.458"/>
-<pinref part="R14" gate="G$1" pin="2"/>
-<pinref part="R15" gate="G$1" pin="2"/>
-<pinref part="+3V16" gate="G$1" pin="+3V3"/>
-</segment>
-</net>
+</net>

Commit message: update
Connections:
- removed net +3V3: C15.1, LUXRGB.VDD
- net VCC: now also C15.1, LUXRGB.VDD
Changed lines of the file:
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@@
 <part name="U$3" library="microbuilder" deviceset="GND" device=""/>
 <part name="C15" library="adafruit" deviceset="C-US" device="C0805" value="0.1uF"/>
-<part name="+3V8" library="supply1" deviceset="+3V3" device=""/>
 <part name="N1" library="con-lstb" deviceset="MA08-1" device=""/>
 <part name="P+11" library="supply1" deviceset="VCC" device=""/>
@@
 <part name="IRG" library="SparkFun-Connectors" deviceset="M01" device="PTH"/>
 <part name="P+3" library="supply1" deviceset="VCC" device=""/>
+<part name="P+4" library="supply1" deviceset="VCC" device=""/>
 </parts>
 <sheets>
@@
 <instance part="U$3" gate="G$1" x="364.236" y="-56.388"/>
 <instance part="C15" gate="G$1" x="399.796" y="-23.368"/>
-<instance part="+3V8" gate="G$1" x="364.236" y="9.652"/>
 <instance part="N1" gate="1" x="416.306" y="133.35"/>
 <instance part="P+11" gate="VCC" x="486.664" y="143.51"/>
@@
 <instance part="IRG" gate="G$1" x="226.06" y="109.22"/>
 <instance part="P+3" gate="VCC" x="304.8" y="101.854"/>
+<instance part="P+4" gate="VCC" x="364.236" y="7.366"/>
 </instances>
 <busses>
@@
 <wire x1="305.054" y1="96.52" x2="305.054" y2="90.678" width="0.1524" layer="91"/>
 </segment>
+<segment>
+<pinref part="LUXRGB" gate="G$1" pin="VDD"/>
+<wire x1="374.396" y1="-33.528" x2="364.236" y2="-33.528" width="0.1524" layer="91"/>
+<wire x1="364.236" y1="-33.528" x2="364.236" y2="2.032" width="0.1524" layer="91"/>
+<wire x1="364.236" y1="2.032" x2="399.796" y2="2.032" width="0.1524" layer="91"/>
+<wire x1="399.796" y1="2.032" x2="399.796" y2="-20.828" width="0.1524" layer="91"/>
+<pinref part="C15" gate="G$1" pin="1"/>
+<wire x1="364.236" y1="2.032" x2="364.236" y2="4.826" width="0.1524" layer="91"/>
+<pinref part="P+4" gate="VCC" pin="VCC"/>
+</segment>
 </net>
 <net name="AREF" class="0">
@@
 </segment>
 </net>
-<net name="+3V3" class="0">
-<segment>
-<pinref part="LUXRGB" gate="G$1" pin="VDD"/>
-<wire x1="374.396" y1="-33.528" x2="364.236" y2="-33.528" width="0.1524" layer="91"/>
-<wire x1="364.236" y1="-33.528" x2="364.236" y2="2.032" width="0.1524" layer="91"/>
-<wire x1="364.236" y1="2.032" x2="364.236" y2="7.112" width="0.1524" layer="91"/>
-<wire x1="364.236" y1="2.032" x2="399.796" y2="2.032" width="0.1524" layer="91"/>
-<wire x1="399.796" y1="2.032" x2="399.796" y2="-20.828" width="0.1524" layer="91"/>
-<junction x="364.236" y="2.032"/>
-<pinref part="C15" gate="G$1" pin="1"/>
-<pinref part="+3V8" gate="G$1" pin="+3V3"/>
-</segment>
-</net>
