File: REVC/open-lux-C.brd (EAGLE design)
At the start: 52.4 x 52.7 mm, 56 parts, among them IC2 MCP73831, IC3 ATMEGA32U4-AU, IC4 MCP1700-33, J1 AYZ0202, Q4 BSS123, T1 FDN340P, T2 FDN340P, T3 FDN340P, X2 USBSMD, X3 8MHz

Commit message: update
Parts:
- removed N1, SV2: (no value), con-lstb:MA08-1
- removed T3: FDN340P, zetex:SOT-23
- removed U$12, U$13, U$14, U$15: WS2813, adafruit:RGBLED5050_4
- added BKO: M10LOCK, SparkFun-Connectors:1X10_LOCK
- added NKA: (no value), SparkFun-Connectors:1X08_LOCK
- moved T1 65.0 mm to (43.9, 33.5)
- moved T2 57.1 mm to (39.4, 33.5)
- moved U$11 33.6 mm to (45.5, 39.4)
- moved RIR4 16.4 mm to (36.1, 27.1)
- moved Q4 9.20 mm to (8.26, 33.1)
- moved U$10 7.13 mm to (38.9, 39.4)
- moved C3 6.91 mm to (8.38, 23.1)
- moved CHG 5.38 mm to (33.3, 3.17), turned to 270 degrees
- moved C4 5.14 mm to (45.0, 44.2), turned to 180 degrees
- moved RTHM1 4.67 mm to (49.3, 44.5)
- moved IC2 4.58 mm to (19.2, 13.1)
- moved RU1 4.20 mm to (18.3, 7.37)
- moved C2 4.10 mm to (13.5, 20.3)
- moved X3 4.10 mm to (19.3, 19.1)
- moved B3 3.82 mm to (2.54, 36.3)
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Connections:
- removed net A6: B1.1
- removed net A7: B2.1
- removed net A8: B3.1
- removed net D3: N1.3
- removed net N$11: U$13.O, U$14.I
- removed net N$27: U$11.O, U$12.I
- removed net N$9: U$14.O, U$15.I
- removed net P0: T1.3, T2.3, T3.3
- removed net VCC1: T2.1
- removed net VCC2: T1.1
- removed net VCC3: T3.1
- removed net V_LCD: T2.2
- removed net V_LCD1: T1.2
- removed net V_LCD2: T3.2
- new net N$8: NKA.6, T1.1
- net A0: now also BKO.7; no longer SV2.7
- net A1: now also BKO.8; no longer SV2.8
- net A2: now also BKO.9; no longer RTHM1.2, THM1.1
- net A3: now also B2.1
- net A4: now also B1.1
- net A5: now also RTHM1.2, THM1.1
- net D10: now also T2.3
- net D11: now also T1.3
- net D12: now also B3.1
- net D13: now also BKO.10
- net D4: no longer N1.4
- net D5: now also Q4.1; no longer N1.5
- net D6: now also NKA.5
- net D7: now also NKA.4
- net D8: now also NKA.3
- net D9: now also NKA.1; no longer Q4.1
- net GND: now also BKO.1, NKA.2, NKA.8; no longer N1.2, N1.8, SV2.1, U$12.S, U$13.S, U$14.S, U$15.S
- net N$4: now also NKA.7, T2.1; no longer U$13.I
- net RESET: no longer N1.1
- net RXD: now also BKO.3; no longer SV2.3
- net SCL: now also BKO.6; no longer SV2.6
- net SDA: now also BKO.5; no longer SV2.5
- net TXD: now also BKO.4; no longer SV2.4
- net VCC: now also BKO.2, T1.2, T2.2; no longer N1.6, SV2.2, U$12.D, U$13.D, U$14.D, U$15.D
Other:
- board text added: "**OPEN-LUX**"
- board text added: "REVC"
- board text added: "publiclab.org/wiki/open-lux"
- board text removed: "PUBLICLAB.ORG"
