File: REVC/open-lux-C.sch (EAGLE design)
At the start: 56 parts, among them IC2 MCP73831, IC3 ATMEGA32U4-AU, IC4 MCP1700-33, J1 AYZ0202, Q4 BSS123, T1 FDN340P, T2 FDN340P, T3 FDN340P, X2 USBSMD, X3 8MHz

Commit message: update
Parts:
- removed N1, SV2: (no value), con-lstb:MA08-1
- removed T3: FDN340P, zetex:PMOSSOT23
- removed U$12, U$13, U$14, U$15: WS2813, adafruit:WS2813
- added BKO: M10LOCK, SparkFun-Connectors:M10LOCK
- added NKA: (no value), SparkFun-Connectors:M08LOCK
Connections:
- removed net A6: B1.P
- removed net A7: B2.P
- removed net A8: B3.P
- removed net D3: N1.3
- removed net N$11: U$13.OUT, U$14.IN
- removed net N$27: U$11.OUT, U$12.IN
- removed net N$9: U$14.OUT, U$15.IN
- removed net P0: T1.G, T2.G, T3.G
- removed net VCC1: T2.D
- removed net VCC2: T1.D
- removed net VCC3: T3.D
- removed net V_LCD: T2.S
- removed net V_LCD1: T1.S
- removed net V_LCD2: T3.S
- new net N$8: NKA.6, T1.D
- net A0: now also BKO.7; no longer SV2.7
- net A1: now also BKO.8; no longer SV2.8
- net A2: now also BKO.9; no longer RTHM1.2, THM1.1
- net A3: now also B2.P
- net A4: now also B1.P
- net A5: now also RTHM1.2, THM1.1
- net D10: now also T2.G
- net D11: now also T1.G
- net D12: now also B3.P
- net D13: now also BKO.10
- net D4: no longer N1.4
- net D5: now also Q4.G; no longer N1.5
- net D6: now also NKA.5
- net D7: now also NKA.4
- net D8: now also NKA.3
- net D9: now also NKA.1; no longer Q4.G
- net GND: now also BKO.1, NKA.2, NKA.8; no longer N1.2, N1.8, SV2.1, U$12.VS, U$13.VS, U$14.VS, U$15.VS
- net N$4: now also NKA.7, T2.D; no longer U$13.IN
- net RESET: no longer N1.1
- net RXD: now also BKO.3; no longer SV2.3
- net SCL: now also BKO.6; no longer SV2.6
- net SDA: now also BKO.5; no longer SV2.5
- net TXD: now also BKO.4; no longer SV2.4
- net VCC: now also BKO.2, T1.S, T2.S; no longer N1.6, SV2.2, U$12.VD, U$13.VD, U$14.VD, U$15.VD
Other:
- note removed: "use high-side switch so that don't need to have two types of mosfets on hand in production?"
- moved on the sheet: B1, B2, T1, T2
