File: REVE/open-lux-E.sch (EAGLE design)
At the start: 54 parts, among them IC1 24AA128SN, IC2 MCP73831, IC3 ATMEGA32U4-AU, IC4 MCP1700-33, J1 AYZ0202, Q4 BSS123, T1 FDN340P, T2 FDN340P, X2 USBSMD, X3 8MHz

Commit message: update
Parts:
- renumbered IC1 to EEPRM
Changed lines of the file:
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@@
 <part name="P+9" library="supply1" deviceset="VCC" device=""/>
 <part name="JP2" library="SparkFun-Connectors" deviceset="M08" device="LOCK"/>
-<part name="IC1" library="microchip" deviceset="24*" device="SN" technology="AA128" value="24AA128SN"/>
+<part name="EEPRM" library="microchip" deviceset="24*" device="SN" technology="AA128" value="24AA128SN"/>
 <part name="GND6" library="supply1" deviceset="GND" device=""/>
 <part name="P+10" library="supply1" deviceset="VCC" device=""/>
@@
 <instance part="P+9" gate="VCC" x="543.814" y="47.498"/>
 <instance part="JP2" gate="G$1" x="297.18" y="147.32"/>
-<instance part="IC1" gate="G$1" x="223.52" y="-74.93"/>
+<instance part="EEPRM" gate="G$1" x="223.52" y="-74.93"/>
 <instance part="GND6" gate="1" x="231.14" y="-88.9"/>
 <instance part="P+10" gate="VCC" x="231.14" y="-57.15"/>
@@
 </segment>
 <segment>
-<pinref part="IC1" gate="G$1" pin="GND"/>
+<pinref part="EEPRM" gate="G$1" pin="GND"/>
 <pinref part="GND6" gate="1" pin="GND"/>
 <wire x1="231.14" y1="-86.36" x2="231.14" y2="-85.09" width="0.1524" layer="91"/>
-<pinref part="IC1" gate="G$1" pin="A2"/>
-<pinref part="IC1" gate="G$1" pin="A1"/>
+<pinref part="EEPRM" gate="G$1" pin="A2"/>
+<pinref part="EEPRM" gate="G$1" pin="A1"/>
 <wire x1="210.82" y1="-74.93" x2="210.82" y2="-77.47" width="0.1524" layer="91"/>
-<pinref part="IC1" gate="G$1" pin="A0"/>
+<pinref part="EEPRM" gate="G$1" pin="A0"/>
 <wire x1="210.82" y1="-77.47" x2="210.82" y2="-80.01" width="0.1524" layer="91"/>
 <junction x="210.82" y="-77.47"/>
@@
 <wire x1="210.82" y1="-86.36" x2="231.14" y2="-86.36" width="0.1524" layer="91"/>
 <junction x="231.14" y="-86.36"/>
-<pinref part="IC1" gate="G$1" pin="WP"/>
+<pinref part="EEPRM" gate="G$1" pin="WP"/>
 <wire x1="210.82" y1="-69.85" x2="210.82" y2="-74.93" width="0.1524" layer="91"/>
 <junction x="210.82" y="-74.93"/>
@@
 </segment>
 <segment>
-<pinref part="IC1" gate="G$1" pin="VCC"/>
+<pinref part="EEPRM" gate="G$1" pin="VCC"/>
 <pinref part="P+10" gate="VCC" pin="VCC"/>
 <wire x1="231.14" y1="-59.69" x2="231.14" y2="-62.23" width="0.1524" layer="91"/>
@@
 </segment>
 <segment>
-<pinref part="IC1" gate="G$1" pin="SDA"/>
+<pinref part="EEPRM" gate="G$1" pin="SDA"/>
 <wire x1="238.76" y1="-74.93" x2="240.538" y2="-74.93" width="0.1524" layer="91"/>
 <label x="240.538" y="-74.168" size="1.778" layer="95"/>
@@
 </segment>
 <segment>
-<pinref part="IC1" gate="G$1" pin="SCL"/>
+<pinref part="EEPRM" gate="G$1" pin="SCL"/>
 <wire x1="210.82" y1="-67.31" x2="207.518" y2="-67.31" width="0.1524" layer="91"/>
 <label x="207.01" y="-66.548" size="1.778" layer="95"/>
