File: REVI/open-lux-I.sch (EAGLE design)
At the start: 54 parts, among them IC2 MCP73831, IC3 ATMEGA32U4-AU, IC4 MCP1700-33, J1 AYZ0202, Q4 BSS123, T1 FDN340P, T2 FDN340P, X2 USBSMD, X3 8MHz

Commit message: update
Parts:
- removed BLNK: 0805, led:LEDCHIPLED_0805
- removed C5: 0.1uF, adafruit:C-USC0805
- removed RE2: 1.5K, rcl:R-EU_R0805
- added LED1, LED2: (no value), adafruit:LEDCHIP-LED0603
- added Q1, Q2: BSS123, transistor-small-signal:BSS123
- added RE3, RE4: 1.5K, rcl:R-EU_R0805
- JP1: value M09 -> (none); device SparkFun-Connectors:M09 -> SparkFun-Connectors:M05LOCK
Connections:
- removed net N$18: BLNK.A, RE2.1
- new net GND1: Q1.S
- new net GND2: Q2.S
- new net N$11: LED1.A, RE3.1
- new net N$12: LED2.C, Q2.D
- new net N$13: LED2.A, RE4.1
- new net N$9: LED1.C, Q1.D
- net A0: now also NKA.5; no longer JP1.8
- net A1: now also NKA.4; no longer JP1.9
- net A2: now also NKA.3
- net A3: now also NKA.1; no longer B2.P
- net A4: now also B2.P; no longer B1.P
- net D12: now also Q1.G; no longer B3.P
- net D13: no longer RE2.2
- net D6: now also Q2.G; no longer NKA.5
- net D7: no longer NKA.4
- net D8: now also B1.P; no longer NKA.3
- net D9: now also B3.P; no longer NKA.1
- net GND: no longer BLNK.C, C5.2
- net SCL: no longer JP1.7
- net SDA: no longer JP1.6
- net VCC: now also RE3.2, RE4.2; no longer C5.1
Other:
- moved on the sheet: LUXNIR1, LUXRGB2
