File: REVM/open-lux-m.brd (EAGLE design)
At the start: 55.7 x 58.5 mm, 65 parts, among them IC2 MCP73831, IC3 ATMEGA32U4-AU, IC4 MCP1700-33, J1 AYZ0202, Q1 BSS123, Q4 BSS123, T3 FDN340P, T4 FDN340P, X2 USBSMD, X3 8MHz

Commit message: update
Parts:
- moved Q4 42.4 mm to (15.2, 44.4)
- moved T4 18.7 mm to (28.3, 30.2)
- moved T3 16.6 mm to (26.6, 32.5)
- moved JP1 2.17 mm to (23.8, 1.58)
- moved RIR3 1.95 mm to (13.9, 47.6), turned to 180 degrees
- moved C7 1.12 mm to (15.1, 30.7)
- moved RE3 0.88 mm to (38.1, 43.1)
- moved IRA 0.82 mm to (11.2, 34.6)
- moved IRP 0.82 mm to (8.63, 37.2)
- moved IRG 0.82 mm to (11.2, 40.0)
- moved IRL 0.82 mm to (13.7, 36.9)
- moved IC3 0.57 mm to (14.1, 18.2), turned to 45 degrees
- moved X3 0.52 mm to (10.4, 30.0)
- moved NKA2 0.49 mm to (36.2, 47.4)
- moved RIR4 0.26 mm to (9.99, 46.5)
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