File: REVN/open-lux-N.sch (EAGLE design)
At the start: 71 parts, among them IC2 MCP73831, IC3 ATMEGA32U4-AU, IC4 MCP1700-33, J1 AYZ0202, Q1 BSS123, Q4 BSS123, T1 FDN340P, T2 FDN340P, X2 USBSMD, X3 8MHz

Commit message: update
Parts:
- removed J1: AYZ0202, SparkFunNew:AYZ0202
- added J2: EG1206, adafruit:EG1206
Connections:
- removed net N$1: J1.1, J1.4
- new net N$16: J2.P
- net VBAT: no longer J1.2, J1.5
- net VDD: now also J2.S; no longer J1.3, J1.6
Other:
- moved on the sheet: IR5
Changed lines of the file:
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@@
 <clearance class="0" value="0.2032"/>
 </class>
-<class number="1" name="power" width="0.254" drill="0">
+<class number="1" name="power" width="0.8128" drill="0">
 <clearance class="1" value="0.2032"/>
 </class>
@@
 <part name="BAT1" library="SparkFunNew" deviceset="BATTERY" device="BATTCOM_20MM_PTH_SMT" value="LIR2032"/>
 <part name="CN1" library="adafruit" deviceset="JST_2PIN" device="-SMT-RA"/>
-<part name="J1" library="SparkFunNew" deviceset="AYZ0202" device=""/>
 <part name="IC4" library="adafruit" deviceset="MCP1700" device="SOT233" value="MCP1700-33"/>
 <part name="C3" library="resistor" deviceset="C-EU" device="C0805" value="10u"/>
@@
 <part name="U$6" library="microbuilder" deviceset="GND" device=""/>
 <part name="U$7" library="SparkFun-Connectors" deviceset="M04X2" device=""/>
+<part name="J2" library="adafruit" deviceset="EG1206" device=""/>
 </parts>
 <sheets>
@@
 </instance>
 <instance part="CN1" gate="G$1" x="102.87" y="91.44"/>
-<instance part="J1" gate="G$1" x="48.26" y="116.84" smashed="yes">
-<attribute name="NAME" x="45.72" y="124.968" size="1.778" layer="95"/>
-</instance>
 <instance part="IC4" gate="1" x="64.77" y="113.03" smashed="yes">
 <attribute name="NAME" x="62.23" y="119.38" size="1.778" layer="95"/>
@@
 </instance>
 <instance part="IR4" gate="G$1" x="153.162" y="134.366"/>
-<instance part="RE5" gate="G$1" x="153.162" y="145.034" smashed="yes" rot="R90">
-<attribute name="NAME" x="151.892" y="147.3454" size="1.778" layer="95" rot="R180"/>
-<attribute name="VALUE" x="149.352" y="144.526" size="1.778" layer="96" rot="R180"/>
+<instance part="RE5" gate="G$1" x="153.162" y="145.288" smashed="yes" rot="R90">
+<attribute name="NAME" x="151.892" y="147.5994" size="1.778" layer="95" rot="R180"/>
+<attribute name="VALUE" x="149.352" y="144.78" size="1.778" layer="96" rot="R180"/>
 </instance>
 <instance part="WS6" gate="G$1" x="129.54" y="196.85"/>
@@
 <instance part="WS9" gate="G$1" x="60.96" y="196.85"/>
 <instance part="WS10" gate="G$1" x="36.83" y="196.85"/>
-<instance part="IR5" gate="G$1" x="163.322" y="134.366"/>
+<instance part="IR5" gate="G$1" x="163.322" y="134.874"/>
 <instance part="RE6" gate="G$1" x="163.322" y="145.034" smashed="yes" rot="R90">
 <attribute name="NAME" x="162.052" y="147.3454" size="1.778" layer="95" rot="R180"/>
@@
 <instance part="U$6" gate="G$1" x="282.194" y="-23.114"/>
 <instance part="U$7" gate="G$1" x="280.67" y="120.396"/>
+<instance part="J2" gate="G$1" x="49.53" y="139.7" smashed="yes" rot="R270">
+<attribute name="NAME" x="47.625" y="136.525" size="1.778" layer="95"/>
+</instance>
 </instances>
 <busses>
@@
 <net name="VDD" class="0">
 <segment>
-<pinref part="J1" gate="G$1" pin="3"/>
-<pinref part="J1" gate="G$1" pin="6"/>
-<wire x1="53.34" y1="116.84" x2="53.34" y2="113.03" width="0.1524" layer="91"/>
 <pinref part="C2" gate="G$1" pin="1"/>
-<wire x1="53.34" y1="113.03" x2="53.34" y2="109.22" width="0.1524" layer="91"/>
-<wire x1="53.34" y1="113.03" x2="57.15" y2="113.03" width="0.1524" layer="91"/>
+<wire x1="52.578" y1="111.76" x2="57.15" y2="113.03" width="0.1524" layer="91"/>
 <wire x1="57.15" y1="113.03" x2="57.15" y2="105.41" width="0.1524" layer="91"/>
-<junction x="53.34" y="113.03"/>
 <pinref part="IC4" gate="1" pin="IN"/>
 <junction x="57.15" y="113.03"/>
+<wire x1="53.848" y1="128.016" x2="52.578" y2="111.76" width="0.1524" layer="91"/>
+<pinref part="J2" gate="G$1" pin="S"/>
+<wire x1="53.848" y1="128.016" x2="54.61" y2="137.16" width="0.1524" layer="91"/>
 </segment>
 </net>
@@
 <pinref part="IC2" gate="G$1" pin="VBAT"/>
 <pinref part="BAT1" gate="G$1" pin="+"/>
-<pinref part="J1" gate="G$1" pin="2"/>
-<wire x1="43.18" y1="119.38" x2="43.18" y2="115.57" width="0.1524" layer="91"/>
-<pinref part="J1" gate="G$1" pin="5"/>
-<wire x1="43.18" y1="115.57" x2="43.18" y2="111.76" width="0.1524" layer="91"/>
-<junction x="43.18" y="115.57"/>
 </segment>
 <segment>
@@
 <pinref part="IC2" gate="G$1" pin="PROG"/>
 <pinref part="RC" gate="G$1" pin="2"/>
-</segment>
-</net>
-<net name="N$1" class="0">
-<segment>
-<pinref part="J1" gate="G$1" pin="1"/>
-<wire x1="53.34" y1="121.92" x2="54.61" y2="121.92" width="0.1524" layer="91"/>
-<wire x1="54.61" y1="121.92" x2="54.61" y2="114.3" width="0.1524" layer="91"/>
-<pinref part="J1" gate="G$1" pin="4"/>
-<wire x1="54.61" y1="114.3" x2="53.34" y2="114.3" width="0.1524" layer="91"/>
 </segment>
 </net>
@@
 <pinref part="RE5" gate="G$1" pin="2"/>
 <wire x1="142.748" y1="155.448" x2="153.162" y2="155.448" width="0.1524" layer="91"/>
-<wire x1="153.162" y1="155.448" x2="153.162" y2="150.114" width="0.1524" layer="91"/>
+<wire x1="153.162" y1="155.448" x2="153.162" y2="150.368" width="0.1524" layer="91"/>
 </segment>
 <segment>
@@
 <pinref part="IR4" gate="G$1" pin="A"/>
 <pinref part="RE5" gate="G$1" pin="1"/>
-<wire x1="153.162" y1="139.954" x2="153.162" y2="136.906" width="0.1524" layer="91"/>
+<wire x1="153.162" y1="140.208" x2="153.162" y2="136.906" width="0.1524" layer="91"/>
 </segment>
 </net>
@@
 <segment>
 <pinref part="IR5" gate="G$1" pin="C"/>
-<wire x1="163.322" y1="129.286" x2="163.322" y2="128.778" width="0.1524" layer="91"/>
-<wire x1="163.322" y1="128.778" x2="163.322" y2="128.524" width="0.1524" layer="91"/>
 <wire x1="152.908" y1="124.714" x2="163.322" y2="124.714" width="0.1524" layer="91"/>
-<wire x1="163.322" y1="124.714" x2="163.322" y2="128.524" width="0.1524" layer="91"/>
+<wire x1="163.322" y1="124.714" x2="163.322" y2="129.794" width="0.1524" layer="91"/>
 </segment>
 </net>
@@
 <pinref part="IR5" gate="G$1" pin="A"/>
 <pinref part="RE6" gate="G$1" pin="1"/>
-<wire x1="163.322" y1="139.954" x2="163.322" y2="136.906" width="0.1524" layer="91"/>
+<wire x1="163.322" y1="139.954" x2="163.322" y2="137.414" width="0.1524" layer="91"/>
 </segment>
 </net>
@@
 </segment>
 </net>
+<net name="N$16" class="1">
+<segment>
+<wire x1="44.45" y1="139.7" x2="43.942" y2="125.73" width="0.1524" layer="91"/>
+<pinref part="J2" gate="G$1" pin="P"/>
+<wire x1="43.434" y1="115.57" x2="43.942" y2="125.73" width="0.1524" layer="91"/>
+</segment>
+</net>

Commit message: update
Parts:
- removed RE2, RE3, RE5, RE6: 1.5K, rcl:R-EU_R0805
- added IRR1, IRR2, IRR4, IRR5: 1.5K, rcl:R-EU_R0805
- renumbered RE4 to IRR3
Connections:
- removed net N$8: IR5.C
- removed net VCC1: RE6.2
- net N$11: now also IRR1.1; no longer RE3.1
- net N$13: now also IRR2.1; no longer RE2.1
- net N$17: now also IRR4.1; no longer RE5.1
- net N$18: now also IRR5.1; no longer RE6.1
- net N$9: now also IR5.C
- net VCC: now also IRR1.2, IRR2.2, IRR4.2, IRR5.2; no longer RE2.2, RE3.2, RE5.2
Changed lines of the file:
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@@
 <setting verticaltext="up"/>
 </settings>
-<grid distance="0.01" unitdist="inch" unit="inch" style="lines" multiple="1" display="no" altdistance="0.01" altunitdist="inch" altunit="inch"/>
+<grid distance="0.1" unitdist="inch" unit="inch" style="lines" multiple="1" display="no" altdistance="0.01" altunitdist="inch" altunit="inch"/>
 <layers>
 <layer number="1" name="Top" color="4" fill="1" visible="no" active="no"/>
@@
 <part name="IR1" library="adafruit" deviceset="LED" device="CHIP-LED0603"/>
 <part name="P+12" library="supply1" deviceset="VCC" device=""/>
-<part name="RE3" library="rcl" deviceset="R-EU_" device="R0805" value="1.5K"/>
+<part name="IRR1" library="rcl" deviceset="R-EU_" device="R0805" value="1.5K"/>
 <part name="LUXNIR1" library="microbuilder" deviceset="TSL2561" device="" value="TSL2561"/>
 <part name="U$3" library="microbuilder" deviceset="GND" device=""/>
@@
 <part name="GND10" library="supply1" deviceset="GND" device=""/>
 <part name="IR2" library="adafruit" deviceset="LED" device="CHIP-LED0603"/>
-<part name="RE2" library="rcl" deviceset="R-EU_" device="R0805" value="1.5K"/>
+<part name="IRR2" library="rcl" deviceset="R-EU_" device="R0805" value="1.5K"/>
 <part name="IR3" library="adafruit" deviceset="LED" device="CHIP-LED0603"/>
-<part name="RE4" library="rcl" deviceset="R-EU_" device="R0805" value="1.5K"/>
+<part name="IRR3" library="rcl" deviceset="R-EU_" device="R0805" value="1.5K"/>
 <part name="IR4" library="adafruit" deviceset="LED" device="CHIP-LED0603"/>
-<part name="RE5" library="rcl" deviceset="R-EU_" device="R0805" value="1.5K"/>
+<part name="IRR4" library="rcl" deviceset="R-EU_" device="R0805" value="1.5K"/>
 <part name="WS6" library="adafruit" deviceset="WS2813" device=""/>
 <part name="WS5" library="adafruit" deviceset="WS2813" device=""/>
@@
 <part name="WS10" library="adafruit" deviceset="WS2813" device=""/>
 <part name="IR5" library="adafruit" deviceset="LED" device="CHIP-LED0603"/>
-<part name="RE6" library="rcl" deviceset="R-EU_" device="R0805" value="1.5K"/>
+<part name="IRR5" library="rcl" deviceset="R-EU_" device="R0805" value="1.5K"/>
 <part name="C9" library="adafruit" deviceset="C-US" device="C0805" value="0.1uF"/>
 <part name="P+20" library="supply1" deviceset="VCC" device=""/>
@@
 <instance part="IR1" gate="G$1" x="117.856" y="134.62"/>
 <instance part="P+12" gate="VCC" x="117.856" y="162.052"/>
-<instance part="RE3" gate="G$1" x="117.856" y="145.288" smashed="yes" rot="R90">
-<attribute name="NAME" x="116.586" y="147.5994" size="1.778" layer="95" rot="R180"/>
-<attribute name="VALUE" x="114.046" y="144.78" size="1.778" layer="96" rot="R180"/>
+<instance part="IRR1" gate="G$1" x="117.856" y="144.272" smashed="yes" rot="R90">
+<attribute name="NAME" x="116.586" y="146.5834" size="1.778" layer="95" rot="R180"/>
+<attribute name="VALUE" x="114.046" y="143.764" size="1.778" layer="96" rot="R180"/>
 </instance>
 <instance part="LUXNIR1" gate="G$1" x="391.414" y="-33.274"/>
@@
 <instance part="GND10" gate="1" x="117.856" y="106.172" rot="MR0"/>
 <instance part="IR2" gate="G$1" x="131.572" y="134.366"/>
-<instance part="RE2" gate="G$1" x="131.572" y="145.034" smashed="yes" rot="R90">
-<attribute name="NAME" x="130.302" y="147.3454" size="1.778" layer="95" rot="R180"/>
-<attribute name="VALUE" x="127.762" y="144.526" size="1.778" layer="96" rot="R180"/>
+<instance part="IRR2" gate="G$1" x="131.572" y="144.526" smashed="yes" rot="R90">
+<attribute name="NAME" x="130.302" y="146.8374" size="1.778" layer="95" rot="R180"/>
+<attribute name="VALUE" x="127.762" y="144.018" size="1.778" layer="96" rot="R180"/>
 </instance>
 <instance part="IR3" gate="G$1" x="142.748" y="134.366"/>
-<instance part="RE4" gate="G$1" x="142.748" y="145.034" smashed="yes" rot="R90">
+<instance part="IRR3" gate="G$1" x="142.748" y="145.034" smashed="yes" rot="R90">
 <attribute name="NAME" x="141.478" y="147.3454" size="1.778" layer="95" rot="R180"/>
 <attribute name="VALUE" x="138.938" y="144.526" size="1.778" layer="96" rot="R180"/>
 </instance>
 <instance part="IR4" gate="G$1" x="153.162" y="134.366"/>
-<instance part="RE5" gate="G$1" x="153.162" y="145.288" smashed="yes" rot="R90">
-<attribute name="NAME" x="151.892" y="147.5994" size="1.778" layer="95" rot="R180"/>
-<attribute name="VALUE" x="149.352" y="144.78" size="1.778" layer="96" rot="R180"/>
+<instance part="IRR4" gate="G$1" x="153.162" y="145.034" smashed="yes" rot="R90">
+<attribute name="NAME" x="151.892" y="147.3454" size="1.778" layer="95" rot="R180"/>
+<attribute name="VALUE" x="149.352" y="144.526" size="1.778" layer="96" rot="R180"/>
 </instance>
 <instance part="WS6" gate="G$1" x="129.54" y="196.85"/>
@@
 <instance part="WS10" gate="G$1" x="36.83" y="196.85"/>
 <instance part="IR5" gate="G$1" x="163.322" y="134.874"/>
-<instance part="RE6" gate="G$1" x="163.322" y="145.034" smashed="yes" rot="R90">
-<attribute name="NAME" x="162.052" y="147.3454" size="1.778" layer="95" rot="R180"/>
-<attribute name="VALUE" x="159.512" y="144.526" size="1.778" layer="96" rot="R180"/>
+<instance part="IRR5" gate="G$1" x="163.322" y="145.542" smashed="yes" rot="R90">
+<attribute name="NAME" x="162.052" y="147.8534" size="1.778" layer="95" rot="R180"/>
+<attribute name="VALUE" x="159.512" y="145.034" size="1.778" layer="96" rot="R180"/>
 </instance>
 <instance part="C9" gate="G$1" x="282.194" y="-7.874"/>
@@
 </segment>
 <segment>
-<pinref part="RE3" gate="G$1" pin="2"/>
+<pinref part="IRR1" gate="G$1" pin="2"/>
 <pinref part="P+12" gate="VCC" pin="VCC"/>
 <wire x1="117.856" y1="159.512" x2="117.856" y2="155.448" width="0.1524" layer="91"/>
-<pinref part="RE2" gate="G$1" pin="2"/>
-<wire x1="117.856" y1="155.448" x2="117.856" y2="150.368" width="0.1524" layer="91"/>
+<pinref part="IRR2" gate="G$1" pin="2"/>
+<wire x1="117.856" y1="155.448" x2="117.856" y2="149.352" width="0.1524" layer="91"/>
 <wire x1="117.856" y1="155.448" x2="131.572" y2="155.448" width="0.1524" layer="91"/>
-<wire x1="131.572" y1="155.448" x2="131.572" y2="150.114" width="0.1524" layer="91"/>
-<pinref part="RE4" gate="G$1" pin="2"/>
+<wire x1="131.572" y1="155.448" x2="131.572" y2="149.606" width="0.1524" layer="91"/>
+<pinref part="IRR3" gate="G$1" pin="2"/>
 <wire x1="131.572" y1="155.448" x2="142.748" y2="155.448" width="0.1524" layer="91"/>
 <wire x1="142.748" y1="155.448" x2="142.748" y2="150.114" width="0.1524" layer="91"/>
-<pinref part="RE5" gate="G$1" pin="2"/>
+<pinref part="IRR4" gate="G$1" pin="2"/>
 <wire x1="142.748" y1="155.448" x2="153.162" y2="155.448" width="0.1524" layer="91"/>
-<wire x1="153.162" y1="155.448" x2="153.162" y2="150.368" width="0.1524" layer="91"/>
+<wire x1="153.162" y1="155.448" x2="153.162" y2="150.114" width="0.1524" layer="91"/>
+<junction x="131.572" y="155.448"/>
+<junction x="142.748" y="155.448"/>
+<pinref part="IRR5" gate="G$1" pin="2"/>
+<wire x1="152.908" y1="155.448" x2="153.162" y2="155.448" width="0.1524" layer="91"/>
+<wire x1="153.162" y1="155.448" x2="163.322" y2="155.448" width="0.1524" layer="91"/>
+<wire x1="163.322" y1="155.448" x2="163.322" y2="150.622" width="0.1524" layer="91"/>
+<junction x="153.162" y="155.448"/>
 </segment>
 <segment>
@@
 <wire x1="142.748" y1="124.714" x2="153.162" y2="124.714" width="0.1524" layer="91"/>
 <wire x1="153.162" y1="124.714" x2="153.162" y2="128.524" width="0.1524" layer="91"/>
+<pinref part="IR5" gate="G$1" pin="C"/>
+<wire x1="152.908" y1="124.714" x2="153.162" y2="124.714" width="0.1524" layer="91"/>
+<wire x1="153.162" y1="124.714" x2="163.322" y2="124.714" width="0.1524" layer="91"/>
+<wire x1="163.322" y1="124.714" x2="163.322" y2="129.794" width="0.1524" layer="91"/>
+<junction x="153.162" y="124.714"/>
+<junction x="142.748" y="124.714"/>
+<junction x="131.572" y="124.714"/>
 </segment>
 </net>
@@
 <segment>
 <pinref part="IR1" gate="G$1" pin="A"/>
-<pinref part="RE3" gate="G$1" pin="1"/>
-<wire x1="117.856" y1="140.208" x2="117.856" y2="137.16" width="0.1524" layer="91"/>
+<pinref part="IRR1" gate="G$1" pin="1"/>
+<wire x1="117.856" y1="139.192" x2="117.856" y2="137.16" width="0.1524" layer="91"/>
 </segment>
 </net>
@@
 <segment>
 <pinref part="IR2" gate="G$1" pin="A"/>
-<pinref part="RE2" gate="G$1" pin="1"/>
-<wire x1="131.572" y1="139.954" x2="131.572" y2="136.906" width="0.1524" layer="91"/>
+<pinref part="IRR2" gate="G$1" pin="1"/>
+<wire x1="131.572" y1="139.446" x2="131.572" y2="136.906" width="0.1524" layer="91"/>
 </segment>
 </net>
@@
 <segment>
 <pinref part="IR3" gate="G$1" pin="A"/>
-<pinref part="RE4" gate="G$1" pin="1"/>
+<pinref part="IRR3" gate="G$1" pin="1"/>
 <wire x1="142.748" y1="139.954" x2="142.748" y2="136.906" width="0.1524" layer="91"/>
 </segment>
@@
 <segment>
 <pinref part="IR4" gate="G$1" pin="A"/>
-<pinref part="RE5" gate="G$1" pin="1"/>
-<wire x1="153.162" y1="140.208" x2="153.162" y2="136.906" width="0.1524" layer="91"/>
+<pinref part="IRR4" gate="G$1" pin="1"/>
+<wire x1="153.162" y1="139.954" x2="153.162" y2="136.906" width="0.1524" layer="91"/>
 </segment>
 </net>
@@
 </segment>
 </net>
-<net name="VCC1" class="0">
-<segment>
-<pinref part="RE6" gate="G$1" pin="2"/>
-<wire x1="152.908" y1="155.448" x2="163.322" y2="155.448" width="0.1524" layer="91"/>
-<wire x1="163.322" y1="155.448" x2="163.322" y2="150.114" width="0.1524" layer="91"/>
-</segment>
-</net>
-<net name="N$8" class="0">
-<segment>
-<pinref part="IR5" gate="G$1" pin="C"/>
-<wire x1="152.908" y1="124.714" x2="163.322" y2="124.714" width="0.1524" layer="91"/>
-<wire x1="163.322" y1="124.714" x2="163.322" y2="129.794" width="0.1524" layer="91"/>
-</segment>
-</net>
 <net name="N$18" class="0">
 <segment>
 <pinref part="IR5" gate="G$1" pin="A"/>
-<pinref part="RE6" gate="G$1" pin="1"/>
-<wire x1="163.322" y1="139.954" x2="163.322" y2="137.414" width="0.1524" layer="91"/>
-</segment>
-</net>
+<pinref part="IRR5" gate="G$1" pin="1"/>
+<wire x1="163.322" y1="140.462" x2="163.322" y2="137.414" width="0.1524" layer="91"/>
+</segment>
+</net>

Commit message: update
Parts:
- removed U$7: M04X2, SparkFun-Connectors:M04X2
- added JP2: M05X2NO_SILK, SparkFun-Connectors:M05X2NO_SILK
Connections:
- net VDD renamed N$1
- removed net N$16: J2.P
- net A0: now also JP2.6; no longer NKA.5, NKA1.6
- net A1: now also B2.P, JP2.8; no longer NKA.4, NKA1.5
- net A2: now also B3.P, JP2.10; no longer NKA.3
- net A3: now also B1.P; no longer NKA.1, NKA1.2
- net A4: now also NKA.1, NKA1.2; no longer B2.P
- net D4: now also NKA.3, NKA1.4; no longer U$7.5
- net D8: now also NKA.5, NKA1.6; no longer B1.P
- net D9: now also NKA.4, NKA1.5; no longer B3.P
- net GND: now also JP2.9; no longer U$7.4
- net RXD: now also JP2.2; no longer U$7.8
- net SCL: now also JP2.3; no longer U$7.3
- net SDA: now also JP2.1; no longer U$7.1
- net TXD: now also JP2.4; no longer U$7.6
- net VBAT: now also J2.P
- net VBUS: now also JP2.5; no longer U$7.7
- net VCC: now also JP2.7
Other:
- moved on the sheet: J2, LUXNIR1
