File: REVN/open-lux-N.brd (EAGLE design)
At the start: 53 x 68.6 mm, 71 parts, among them IC2 MCP73831, IC3 ATMEGA32U4-AU, IC4 MCP1700-33, J2 EG1206, Q1 BSS123, Q4 BSS123, T1 FDN340P, T2 FDN340P, X2 USBSMD, X3 8MHz

Commit message: update
Parts:
- moved IRG 1.14 mm to (11.9, 59.2)
- moved IRL 1.14 mm to (9.40, 56.6)
- moved IRP 1.14 mm to (14.5, 56.6)
- moved IRA 1.14 mm to (11.9, 54.1)
Routing:
- net VCC: track 420.0 -> 418.2 mm
- net A2: track 83.2 -> 84.9 mm
- net SCL: track 141.3 -> 139.7 mm
- net VBUS: track 139.8 -> 140.4 mm
Other:
- board text added: "PUBLICLAB.ORG/WIKI/OPEN-LUX"
- board text removed: "HTTP://PUBLICLAB.ORG/WIKI/OPEN-LUX"
