File: REVQ/open-lux-Q.brd (EAGLE design)
At the start: 53 x 68.6 mm, 76 parts, among them IC2 MCP73831, IC3 ATMEGA32U4-AU, IC4 MCP1700-33, J2 EG1206, Q1 BSS123, Q4 BSS123, T1 FDN340P, T2 FDN340P, X2 USBSMD, X3 8MHz

Commit message: update
Parts:
- renumbered J2 to SWITCH, JST to USB
Other:
- board text added: "REV-Q"
- board text added: "VBAT"
- board text removed: "LUXNIR"
- board text removed: "REV-O"
- board text removed: "RGB"
