File: REVQ/rgb-nir-uv-breakout.brd (EAGLE design)
At the start: 19.5 x 18.4 mm, 15 parts, among them U1 ML8511-UV-SENSOR

Commit message: update
Parts:
- removed IRA, IRG, IRL, IRP: M01PTH, SparkFun-Connectors:1X01
- removed RIR3, RIR4: 10K, rcl:R0805
- removed SJ1: SOLDERJUMPERTRACE, SparkFun-Passives:SJ_2S-TRACE
- moved RUV 0.80 mm to (24.4, 12.2), turned to 0 degrees
- moved JP3 0.28 mm to (19.1, 24.1)
Connections:
- removed net N$1: LUXNIR.ADR, SJ1.1
- net GND: no longer IRG.1
- net SCL: no longer IRL.1, RIR3.1
- net SDA: no longer IRA.1, RIR4.1
- net VCC: now also LUXNIR.ADR; no longer IRP.1, RIR3.2, RIR4.2, SJ1.2
Routing:
- net N$1: track 21.6 -> 0.00 mm, vias 2 -> 0
- net ENABLE: track 25.7 -> 13.6 mm
- net SCL: track 22.6 -> 16.2 mm, vias 2 -> 3
- net GND: track 22.0 -> 15.9 mm, vias 1 -> 2
- net VCC: track 41.2 -> 36.5 mm, vias 5 -> 2
- net N$8: track 7.02 -> 11.2 mm, vias 2 -> 0
- net A1: track 24.6 -> 26.0 mm, vias 2 -> 3
- net SDA: track 14.4 -> 15.2 mm
