File: REVQ/rgb-nir-uv-breakout.sch (EAGLE design)
At the start: 15 parts, among them U1 ML8511-UV-SENSOR

Commit message: update
Parts:
- removed IRA, IRG, IRL, IRP: M01PTH, SparkFun-Connectors:M01PTH
- removed RIR3, RIR4: 10K, rcl:R-EU_R0805
- removed SJ1: SOLDERJUMPERTRACE, SparkFun-Passives:SOLDERJUMPERTRACE
Connections:
- removed net N$1: LUXNIR.ADDRSEL, SJ1.1
- net GND: no longer IRG.1
- net SCL: no longer IRL.1, RIR3.1
- net SDA: no longer IRA.1, RIR4.1
- net VCC: now also LUXNIR.ADDRSEL; no longer IRP.1, RIR3.2, RIR4.2, SJ1.2
Changed lines of the file:
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@@
 <part name="C8" library="adafruit" deviceset="C-US" device="C0805" value="1nF"/>
 <part name="RUV" library="rcl" deviceset="R-EU_" device="R0805" value="10K"/>
-<part name="SJ1" library="SparkFun-Passives" deviceset="SOLDERJUMPER" device="TRACE"/>
-<part name="RIR3" library="rcl" deviceset="R-EU_" device="R0805" value="10K"/>
-<part name="RIR4" library="rcl" deviceset="R-EU_" device="R0805" value="10K"/>
-<part name="P+7" library="supply1" deviceset="VCC" device=""/>
-<part name="P+13" library="supply1" deviceset="VCC" device=""/>
-<part name="GND11" library="SparkFun" deviceset="GND" device=""/>
-<part name="IRL" library="SparkFun-Connectors" deviceset="M01" device="PTH"/>
-<part name="IRA" library="SparkFun-Connectors" deviceset="M01" device="PTH"/>
-<part name="IRP" library="SparkFun-Connectors" deviceset="M01" device="PTH"/>
-<part name="IRG" library="SparkFun-Connectors" deviceset="M01" device="PTH"/>
 </parts>
 <sheets>
@@
 <attribute name="VALUE" x="44.45" y="-102.108" size="1.778" layer="96" rot="R180"/>
 </instance>
-<instance part="SJ1" gate="1" x="-29.972" y="-21.336" rot="R90"/>
-<instance part="RIR3" gate="G$1" x="177.8" y="53.34" smashed="yes" rot="R90">
-<attribute name="NAME" x="181.61" y="53.34" size="1.778" layer="95"/>
-<attribute name="VALUE" x="179.07" y="50.8" size="1.778" layer="96"/>
-</instance>
-<instance part="RIR4" gate="G$1" x="182.88" y="40.64" smashed="yes" rot="R90">
-<attribute name="NAME" x="184.15" y="40.64" size="1.778" layer="95"/>
-<attribute name="VALUE" x="184.15" y="38.1" size="1.778" layer="96"/>
-</instance>
-<instance part="P+7" gate="VCC" x="180.34" y="60.96"/>
-<instance part="P+13" gate="VCC" x="210.82" y="38.1"/>
-<instance part="GND11" gate="1" x="210.82" y="12.7"/>
-<instance part="IRL" gate="G$1" x="167.64" y="48.26"/>
-<instance part="IRA" gate="G$1" x="167.64" y="35.56"/>
-<instance part="IRP" gate="G$1" x="195.58" y="27.94"/>
-<instance part="IRG" gate="G$1" x="195.58" y="15.24"/>
 </instances>
 <busses>
@@
 <wire x1="12.7" y1="-124.46" x2="12.7" y2="-127" width="0.1524" layer="91"/>
 <pinref part="C8" gate="G$1" pin="2"/>
-</segment>
-<segment>
-<wire x1="203.2" y1="15.24" x2="210.82" y2="15.24" width="0.1524" layer="91"/>
-<pinref part="GND11" gate="1" pin="GND"/>
-<pinref part="IRG" gate="G$1" pin="1"/>
 </segment>
 </net>
@@
 <wire x1="34.544" y1="-12.954" x2="28.194" y2="-12.954" width="0.1524" layer="91"/>
 <wire x1="34.29" y1="-4.318" x2="34.544" y2="-7.112" width="0.1524" layer="91"/>
-<wire x1="34.544" y1="-7.112" x2="34.29" y2="-9.906" width="0.1524" layer="91"/>
-<wire x1="34.29" y1="-9.906" x2="34.544" y2="-12.954" width="0.1524" layer="91"/>
-<pinref part="SJ1" gate="1" pin="2"/>
-<wire x1="34.29" y1="-9.906" x2="-18.034" y2="-9.906" width="0.1524" layer="91"/>
-<wire x1="-18.034" y1="-9.906" x2="-29.972" y2="-16.256" width="0.1524" layer="91"/>
+<wire x1="34.544" y1="-7.112" x2="34.544" y2="-9.652" width="0.1524" layer="91"/>
+<pinref part="LUXNIR" gate="G$1" pin="ADDRSEL"/>
+<wire x1="34.544" y1="-9.652" x2="34.544" y2="-12.954" width="0.1524" layer="91"/>
+<wire x1="33.274" y1="-25.654" x2="20.32" y2="-25.654" width="0.1524" layer="91"/>
+<wire x1="20.32" y1="-25.654" x2="20.32" y2="-9.652" width="0.1524" layer="91"/>
+<wire x1="20.32" y1="-9.652" x2="34.544" y2="-9.652" width="0.1524" layer="91"/>
 </segment>
 <segment>
@@
 <pinref part="RUV" gate="G$1" pin="2"/>
 </segment>
-<segment>
-<pinref part="RIR4" gate="G$1" pin="2"/>
-<wire x1="182.88" y1="45.72" x2="182.88" y2="58.42" width="0.1524" layer="91"/>
-<pinref part="RIR3" gate="G$1" pin="2"/>
-<wire x1="182.88" y1="58.42" x2="180.34" y2="58.42" width="0.1524" layer="91"/>
-<pinref part="P+7" gate="VCC" pin="VCC"/>
-<wire x1="180.34" y1="58.42" x2="177.8" y2="58.42" width="0.1524" layer="91"/>
-<junction x="180.34" y="58.42"/>
-</segment>
-<segment>
-<wire x1="203.2" y1="27.94" x2="210.82" y2="27.94" width="0.1524" layer="91"/>
-<wire x1="210.82" y1="27.94" x2="210.82" y2="35.56" width="0.1524" layer="91"/>
-<pinref part="P+13" gate="VCC" pin="VCC"/>
-<pinref part="IRP" gate="G$1" pin="1"/>
-</segment>
 </net>
 <net name="A2" class="0">
@@
 <label x="104.394" y="-41.402" size="1.778" layer="95"/>
 </segment>
-<segment>
-<wire x1="175.26" y1="35.56" x2="182.88" y2="35.56" width="0.1524" layer="91"/>
-<pinref part="RIR4" gate="G$1" pin="1"/>
-<pinref part="IRA" gate="G$1" pin="1"/>
-<wire x1="182.88" y1="35.56" x2="193.04" y2="35.56" width="0.1524" layer="91"/>
-<label x="193.04" y="35.56" size="1.778" layer="95"/>
-</segment>
 </net>
 <net name="SCL" class="0">
@@
 <wire x1="124.714" y1="-46.482" x2="104.394" y2="-46.482" width="0.1524" layer="91"/>
 <label x="104.394" y="-46.482" size="1.778" layer="95"/>
-</segment>
-<segment>
-<wire x1="175.26" y1="48.26" x2="177.8" y2="48.26" width="0.1524" layer="91"/>
-<pinref part="RIR3" gate="G$1" pin="1"/>
-<pinref part="IRL" gate="G$1" pin="1"/>
-<wire x1="177.8" y1="48.26" x2="193.04" y2="48.26" width="0.1524" layer="91"/>
-<label x="193.04" y="48.26" size="1.778" layer="95"/>
 </segment>
 </net>
@@
 </segment>
 </net>
-<net name="N$1" class="0">
-<segment>
-<pinref part="LUXNIR" gate="G$1" pin="ADDRSEL"/>
-<wire x1="33.274" y1="-25.654" x2="11.43" y2="-25.654" width="0.1524" layer="91"/>
-<pinref part="SJ1" gate="1" pin="1"/>
-<wire x1="-29.972" y1="-26.416" x2="11.43" y2="-25.654" width="0.1524" layer="91"/>
-</segment>
-</net>
