File: REVT/open-lux-T-fixbutt.brd (EAGLE design)
At the start: 53.9 x 70.9 mm, 68 parts, among them IC1 MCP23008, IC2 MCP73831, IC3 ATMEGA32U4-AU, IC4 MCP1700-33, Q4 BSS123, T1 FDN340P, T2 FDN340P, X2 USBSMD, X3 8MHz

Commit message: update
Parts:
- moved B2 10.7 mm to (50.6, 38.8)
- moved B3 9.83 mm to (50.5, 49.2)
- moved Q4 2.30 mm to (11.7, 34.7)
- moved RD+1 2.13 mm to (35.6, 20.7)
- moved MICROSD 2.08 mm to (46.3, 16.9)
- moved RU1 1.92 mm to (45.2, 20.8)
- moved RD-1 1.35 mm to (40.4, 20.9)
- moved IC2 1.12 mm to (49.6, 19.2)
- moved RN2 0.77 mm to (47.9, 56.2)
- moved IC1 0.76 mm to (47.8, 64.6)
- moved X2 0.64 mm to (47.4, 27.7)
- moved CEXP1 0.52 mm to (52.2, 55.7)
- moved JP4 0.51 mm to (1.37, 30.8)
- moved PWR 0.46 mm to (52.2, 16.6)
- moved U$1 0.34 mm to (12.3, 66.0)
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Routing:
- net N$35: track 65.5 -> 27.8 mm, vias 6 -> 3
- net D12: track 41.0 -> 75.5 mm, vias 5 -> 6
- net SCL: track 164.7 -> 194.5 mm, vias 9 -> 11
- net VCC: track 424.4 -> 398.3 mm, vias 23 -> 19
- net SDA: track 172.8 -> 147.2 mm, vias 9 -> 10
- net MOSI: track 153.3 -> 130.8 mm, vias 8 -> 6
- net MISO: track 120.4 -> 103.6 mm
- net VBUS: track 167.1 -> 150.7 mm, vias 10 -> 7
- net D5: track 30.9 -> 46.5 mm, vias 2 -> 4
- net N$33: track 40.4 -> 24.9 mm
- net RX: track 60.2 -> 75.6 mm, vias 6 -> 5
- net GND: track 491.0 -> 503.1 mm, vias 20 -> 15
- net N$6: track 16.6 -> 28.2 mm, vias 2 -> 0
- net N$14: track 16.9 -> 7.69 mm
- net N$17: track 38.5 -> 29.3 mm, vias 4 -> 2
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