File: REVT/open-lux-T.brd (EAGLE design)
At the start: 53.9 x 70.9 mm, 68 parts, among them IC1 MCP23008, IC2 MCP73831, IC3 ATMEGA32U4-AU, IC4 MCP1700-33, Q4 BSS123, T1 FDN340P, T2 FDN340P, X2 USBSMD, X3 8MHz

Commit message: update
Parts:
- moved JP5 1.44 mm to (33.9, 35.8)
- moved JP6 1.44 mm to (33.9, 46.0)
- moved JP1 1.44 mm to (23.7, 38.4)
- moved JP3 1.44 mm to (23.7, 48.6)
- moved LED6 0.78 mm to (15.6, 53.5)
- moved LED5 0.70 mm to (23.6, 59.4)
- moved RN1 0.64 mm to (28.4, 53.3)
- moved LED4 0.60 mm to (33.6, 59.3)
- moved LED1 0.55 mm to (41.0, 34.5)
- moved LED7 0.54 mm to (12.7, 44.1)
- moved LED8 0.34 mm to (15.9, 34.5)
- moved B3 0.31 mm to (50.1, 39.5)
- moved LED2 0.31 mm to (44.4, 43.8)
- moved C1 0.23 mm to (19.1, 43.9)
- moved WS1 0.16 mm to (20.4, 32.3)
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Routing:
- net N$12: track 16.9 -> 85.0 mm, vias 0 -> 3
- net SDA: track 172.8 -> 138.9 mm, vias 9 -> 8
- net MOSI: track 153.3 -> 123.0 mm, vias 8 -> 6
- net MISO: track 120.4 -> 146.7 mm
- net VCC: track 424.4 -> 402.6 mm, vias 23 -> 27
- net D4: track 52.0 -> 72.4 mm, vias 6 -> 3
- net A2: track 100.0 -> 120.4 mm
- net D10: track 21.6 -> 41.3 mm, vias 1 -> 5
- net A0: track 88.4 -> 104.8 mm, vias 8 -> 7
- net N$35: track 65.5 -> 49.3 mm, vias 6 -> 3
- net D13: track 77.3 -> 61.9 mm, vias 2 -> 4
- net GND: track 491.0 -> 476.7 mm, vias 20 -> 18
- net N$26: track 10.3 -> 21.7 mm, vias 1 -> 2
- net VBAT: track 87.9 -> 98.9 mm, vias 3 -> 7
- net N$29: track 31.8 -> 42.7 mm, vias 2 -> 1
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Other:
- board size 53.9 x 70.9 mm -> 54 x 70.9 mm
- board text added: "publiclab.org/wiki/open-lux"
